File: HW/stm32_timer_app/stm32_timer_app.kicad_pcb (KiCad board)
At the start: 2 copper layers, 161.3 x 76.1 mm, 91 parts, among them IC1 STM32F303C8T6, J1 691213710002, J2 61300411121, J3 691213710002, J4 61300411121, J5 61300411121, J6 61300411121, J7 105164-0001, U1 MOC3041SM, U2 STM32F103C8T6, U3 MAX31865 AMPLIFIER, U4 RT9193-33GB, U5 MMBT2222A-7-F, U6 SMTU2032-LF, Y1 ABM3-8.000MHZ-J4Q-T, Y2 ABS07-32.768KHZ-T

Commit message: final schematic
Parts:
- removed C16, C17: 105, LD03ZD475MAB2A:CAPC1608X90
- removed IC1: STM32F303C8T6, STM32F103C8T6:QFP50P900X900X160-48N
- removed J6: 61300411121, 61300411121:CONN_61300411121_WRE
- removed R21: 330, Resistor_SMD:R_0603_1608Metric
- removed R3: 360, Resistor_SMD:R_0603_1608Metric
- removed S2, S3: 1571527-1, 1571527-1:SW_1571527-1
- added C22: 103, LD03ZD475MAB2A:CAPC1608X90, F.Cu at (170.9, 73.7)
- added C23: 104, LD03ZD475MAB2A:CAPC1608X90, F.Cu at (176.4, 80.0)
- added C24: 103, LD03ZD475MAB2A:CAPC1608X90, F.Cu at (177.8, 69.6)
- added C25: 104, LD03ZD475MAB2A:CAPC1608X90, F.Cu at (180.6, 75.0)
- added J10: 75160-196-03LF, 75160-196-03LF:AMPHENOL_75160-196-03LF, F.Cu at (155.0, 66.7)
- added J8: PH1RB-04-UA, PH1RB-04-UA:HDRRA4W64P0X254_1X4_1016X250X850P, F.Cu at (190.6, 41.4)
- added J9: PH1RB-05-UA_TEMP., PH1RB-05-UA_TEMP:HDRRA5W64P0X254_1X5_1270X250X288P, F.Cu at (187.0, 38.4)
- added REF**: TestPoint_Pad_D1.0mm, TestPoint:TestPoint_Pad_D1.0mm, F.Cu at (193.8, 46.1)
- added REF**: TestPoint_Pad_D1.0mm, TestPoint:TestPoint_Pad_D1.0mm, F.Cu at (174.5, 61.4)
- added REF**: TestPoint_Pad_D1.0mm, TestPoint:TestPoint_Pad_D1.0mm, F.Cu at (180.7, 61.6)
- added REF**: TestPoint_Pad_D1.0mm, TestPoint:TestPoint_Pad_D1.0mm, B.Cu at (163.8, 53.5)
- added REF**: TestPoint_Pad_D1.0mm, TestPoint:TestPoint_Pad_D1.0mm, B.Cu at (170.3, 51.0)
- added REF**: TestPoint_Pad_D1.0mm, TestPoint:TestPoint_Pad_D1.0mm, F.Cu at (175.8, 63.5)
- added REF**: TestPoint_Pad_D1.0mm, TestPoint:TestPoint_Pad_D1.0mm, F.Cu at (215.9, 106.9)
- added REF**: TestPoint_Pad_D1.0mm, TestPoint:TestPoint_Pad_D1.0mm, F.Cu at (190.9, 44.7)
- added TP1: TestPoint_Probe, TestPoint:TestPoint_THTPad_D2.0mm_Drill1.0mm, F.Cu at (164.1, 40.1)
- added TP11: TestPoint_Probe, TestPoint:TestPoint_THTPad_D2.0mm_Drill1.0mm, F.Cu at (221.2, 108.2)
- added TP12: TestPoint_Probe, TestPoint:TestPoint_THTPad_D2.0mm_Drill1.0mm, F.Cu at (167.9, 107.0)
- added TP13: TestPoint_Probe, TestPoint:TestPoint_THTPad_D2.0mm_Drill1.0mm, F.Cu at (201.8, 59.0)
- added TP14: TestPoint_Probe, TestPoint:TestPoint_THTPad_D2.0mm_Drill1.0mm, F.Cu at (200.1, 50.5)
- added TP15: TestPoint_Probe, TestPoint:TestPoint_THTPad_D2.0mm_Drill1.0mm, F.Cu at (201.7, 46.1)
- added TP16: TestPoint_Probe, TestPoint:TestPoint_THTPad_D2.0mm_Drill1.0mm, F.Cu at (198.4, 45.5)
- added TP17: TestPoint_Probe, TestPoint:TestPoint_THTPad_D2.0mm_Drill1.0mm, F.Cu at (209.2, 97.5)
- added TP19: TestPoint_Probe, TestPoint:TestPoint_THTPad_D2.0mm_Drill1.0mm, F.Cu at (250.7, 108.2)
- added TP2: TestPoint_Probe, TestPoint:TestPoint_THTPad_D2.0mm_Drill1.0mm, F.Cu at (153.8, 43.9)
- added TP20: TestPoint_Probe, TestPoint:TestPoint_THTPad_D2.0mm_Drill1.0mm, F.Cu at (255.9, 108.2)
- added TP21: TestPoint_Probe, TestPoint:TestPoint_THTPad_D2.0mm_Drill1.0mm, F.Cu at (268.1, 90.6)
- added TP22: TestPoint_Probe, TestPoint:TestPoint_THTPad_D2.0mm_Drill1.0mm, F.Cu at (267.8, 71.2)
- added TP23: TestPoint_Probe, TestPoint:TestPoint_THTPad_D2.0mm_Drill1.0mm, F.Cu at (268.1, 87.2)
- added TP25: TestPoint_Probe, TestPoint:TestPoint_THTPad_D2.0mm_Drill1.0mm, F.Cu at (157.7, 58.2)
- added TP4: TestPoint_Probe, TestPoint:TestPoint_THTPad_D2.0mm_Drill1.0mm, F.Cu at (208.9, 90.2)
- added TP5: TestPoint_Probe, TestPoint:TestPoint_THTPad_D2.0mm_Drill1.0mm, F.Cu at (237.7, 81.0)
- added TP8: TestPoint_Probe, TestPoint:TestPoint_THTPad_D2.0mm_Drill1.0mm, F.Cu at (244.5, 89.0)
- added U8: MPU-6050, MPU_6050:QFN24_4X4X0P9_IVS, F.Cu at (176.2, 74.9)
- C1, C2, C7, C8, R1, R19, R25, R26: moved to B.Cu
- J5: value 61300411121 -> 54101-G0502LF; footprint 61300411121:CONN_61300411121_WRE -> 54101-G0502LF:AMPHENOL_54101-G0502LF
- R14: moved to F.Cu
- R2: value 1K -> 330; footprint Resistor_SMD:R_0603_1608Metric -> RC1206FR_0728RL:RC1206N_YAG
- R20, R7, R9: footprint Resistor_SMD:R_0603_1608Metric -> RC1206FR_0728RL:RC1206N_YAG
- R8: value 330 -> 1k; footprint Resistor_SMD:R_0603_1608Metric -> RC1206FR_0728RL:RC1206N_YAG
- U2: value STM32F103C8T6 -> STM32F303C8T6
- moved C9 99.3 mm to (205.3, 39.9), turned to -90 degrees
- moved C6 95.7 mm to (208.4, 39.9), turned to -90 degrees
- moved C4 92.2 mm to (211.6, 39.9), turned to -90 degrees
- moved C2 91.7 mm to (200.0, 53.4), turned to 180 degrees
- moved C8 91.3 mm to (196.3, 48.2), turned to 180 degrees
- moved C7 91.1 mm to (196.3, 51.0), turned to 180 degrees
- moved C3 88.7 mm to (214.7, 39.9), turned to -90 degrees
- moved R1 86.9 mm to (202.9, 54.7), turned to -90 degrees
- moved R20 81.0 mm to (131.3, 78.0), turned to -90 degrees
- moved C1 80.7 mm to (200.0, 56.0), turned to 180 degrees
- moved C21 77.1 mm to (208.9, 103.3)
- moved CR2 76.6 mm to (209.3, 100.5)
- moved LED2 74.7 mm to (168.7, 89.8), turned to 0 degrees
- moved R4 74.7 mm to (164.6, 89.8)
- moved C20 42.3 mm to (172.3, 40.0), turned to 90 degrees
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Connections:
- C1 pad 1: Net-(C1-Pad1) -> GND
- C10 pad 1: Net-(U4-GND) -> GND
- C11 pad 1: Net-(U4-GND) -> GND
- C12 pad 1: Net-(U4-GND) -> GND
- C13 pad 1: Net-(C13-Pad1) -> GND
- C14 pad 1: Net-(C14-Pad1) -> GND
- C15 pad 2: Net-(C15-Pad2) -> GND
- C18 pad 1: /PA4 -> /PA13
- C18 pad 2: Net-(C18-Pad2) -> GND
- C19 pad 1: /PA3 -> /PA2
- C19 pad 2: Net-(C19-Pad2) -> GND
- C2 pad 1: Net-(C1-Pad1) -> GND
- C20 pad 2: Net-(C20-Pad2) -> GND
- C21 pad 2: Net-(C21-Pad2) -> GND
- C3 pad 2: Net-(C3-Pad2) -> GND
- C4 pad 2: Net-(C3-Pad2) -> GND
- C6 pad 2: Net-(C3-Pad2) -> GND
- C7 pad 1: Net-(C7-Pad1) -> GND
- C8 pad 1: Net-(C8-Pad1) -> GND
- C9 pad 2: Net-(C3-Pad2) -> GND
- DS1 pad 1: Net-(DS1-GND) -> GND
- DS1 pad 5: /PA6 -> /PB8
- DS1 pad 6: /PB3 -> /PB5
- J2 pad 1: /+3.3VT -> GND
- J2 pad 2: Net-(J2-Pad2) -> /+3.3VT
- J2 pad 3: /PA10T -> /LED
- J4 pad 1: /+3.3V -> GND
- J4 pad 2: Net-(J4-Pad2) -> /+3.3V
- J4 pad 3: /PA10 -> /PB14
- J4 pad 4: /PB7 -> /PB15
- J7 pad 1: Net-(J7-G) -> GND
- J7 pad 2: Net-(J7-G) -> GND
- J7 pad SH1: Net-(J7-SHIELD-PadSH1) -> GND
- J7 pad SH2: Net-(J7-SHIELD-PadSH1) -> GND
- J7 pad SH3: Net-(J7-SHIELD-PadSH1) -> GND
- J7 pad SH4: Net-(J7-SHIELD-PadSH1) -> GND
- J7 pad SH5: Net-(J7-SHIELD-PadSH1) -> GND
- J7 pad SH6: Net-(J7-SHIELD-PadSH1) -> GND
- MT1 pad 1: Net-(MT1-Pad1) -> GND
- MT1 pad 2: /PA2 -> /PA3
- MT1 pad A: /PA0 -> /PA1
- MT1 pad B: /PA1 -> /PA0
- MT1 pad COM: Net-(MT1-Pad1) -> GND
- MT1 pad S1: Net-(MT1-Pad1) -> GND
- MT1 pad S2: Net-(MT1-Pad1) -> GND
- MT2 pad 1: Net-(MT2-Pad1) -> GND
- MT2 pad A: /PB5 -> /PA4
- MT2 pad COM: Net-(MT2-Pad1) -> GND
- MT2 pad S1: Net-(MT2-Pad1) -> GND
- MT2 pad S2: Net-(MT2-Pad1) -> GND
- R11 pad 1: Net-(R11-Pad1) -> GND
- R12 pad 1: /PA1 -> /PA0
- R13 pad 1: /PA0 -> /PA1
- R14 pad 1: /PA2 -> /PA3
- R16 pad 1: /PB5 -> /PA4
- R2 pad 1: Net-(J2-Pad4) -> Net-(D1-Pad3)
- R2 pad 2: Net-(R2-Pad2) -> Net-(C5-Pad1)
- R20 pad 1: /PA8 -> GND
- R20 pad 2: /+3.3V -> Net-(LED4-Pad1)
- R22 pad 1: /PA4 -> /PA13
- R23 pad 1: /PA3 -> /PA2
- R4 pad 1: /PB8 -> /PB12
- R4 pad 2: Net-(LED1-Pad1) -> Net-(LED2-Pad1)
- R6 pad 2: Net-(LED2-Pad1) -> Net-(LED1-Pad1)
- R7 pad 1: Net-(C5-Pad1) -> Net-(D1-Pad1)
- R7 pad 2: Net-(D1-Pad3) -> Net-(R7-Pad2)
- R8 pad 1: /PA10T -> Net-(R8-Pad1)
- R8 pad 2: Net-(LED3-Pad1) -> Net-(J2-Pad4)
- R9 pad 1: Net-(R9-Pad1) -> /LED
- R9 pad 2: Net-(LED4-Pad1) -> Net-(LED3-Pad1)
- S4 pad 2: Net-(S4-Pad2) -> GND
- S5 pad 3: Net-(S5-Pad1) -> GND
- S5 pad 4: /PA4 -> /PA13
- S6 pad 3: Net-(S6-Pad1) -> GND
- S6 pad 4: /PA3 -> /PA2
- S7 pad 3: Net-(S7-Pad3) -> GND
- S8 pad 3: Net-(S8-Pad3) -> GND
- U1 pad 1: Net-(R2-Pad2) -> Net-(R8-Pad1)
- U1 pad 2: Net-(U1-Pad2) -> GND
- U1 pad 6: Net-(R3-Pad1) -> Net-(R7-Pad2)
- U2 pad 1: unconnected-(U2-VBAT-Pad1) -> /VBAT
- U2 pad 23: Net-(U2-VSSA) -> GND
- U2 pad 26: /PB13 -> /PA13
- U2 pad 35: Net-(U2-VSSA) -> GND
- U2 pad 47: Net-(U2-VSSA) -> GND
- U2 pad 8: Net-(U2-VSSA) -> GND
- U3 pad 2: Net-(U3-GND) -> GND
- U3 pad 4: /PB13 -> /PA5
- U3 pad 5: /PB15 -> /PA7
- U3 pad 6: /PB14 -> /PA6
- U3 pad 7: /PB12 -> /PB6
- U4 pad 2: Net-(U4-GND) -> GND
- U5 pad 2: Net-(U5-E) -> GND
- U6 pad 2: Net-(U6--) -> GND
Routing:
- net /+3.3V: track 224.9 -> 519.6 mm, vias 1 -> 3
- net /VBAT: track 0.00 -> 217.0 mm, vias 0 -> 1
- net /PB9: track 0.00 -> 98.4 mm, vias 0 -> 3
- net /PA4: track 9.04 -> 96.9 mm, vias 0 -> 1
- net /PA13: track 0.00 -> 80.9 mm, vias 0 -> 1
- net /PB1: track 0.00 -> 80.4 mm, vias 0 -> 2
- net /BOOT1: track 0.00 -> 79.2 mm, vias 0 -> 2
- net /PB11: track 0.00 -> 65.9 mm, vias 0 -> 1
- net /PA7: track 25.7 -> 86.2 mm
- net /PA5: track 28.2 -> 87.5 mm
- net /PB6: track 33.4 -> 91.7 mm, vias 1 -> 2
- net /PB15: track 0.00 -> 58.3 mm
- net /PB5: track 90.4 -> 32.6 mm
- net /RESET: track 7.18 -> 63.0 mm, vias 0 -> 1
- net /PB12: track 0.00 -> 54.7 mm, vias 0 -> 1
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- added copper zone on B.Cu, net GND
- added copper zone on F.Cu, net GND
Other:
- outline, holes or cut-outs redrawn
- board text added: "+5V"
- board text added: "3v3"
- board text added: "AUX_CL"
- board text added: "AUX_DA"
- board text added: "GND"
- board text added: "LED"
- board text added: "LINE"
- board text added: "MPU6050"
- board text added: "NEUTRAL"
- board text added: "PA11"
- board text added: "PA12"
- board text added: "PA15"
- board text added: "PA8"
- board text added: "PA9"
- board text added: "PB10"
- board text added: "PB7"
- board text added: "Rx"
- board text added: "SIG"
- board text added: "SWDCLK"
- board text added: "SWDIO"
- board text added: "TRAC"
- board text added: "TRIAC DRIVE"
- board text added: "Tx"
- board text added: "USART"
- board text added: "VBAT"
- board text added: "capacitive"
- board text removed: "Button1"
- board text removed: "Button2"
- board text removed: "PINs"
